Commit message: Добавлены плагины, но не настроены

File: plastun_description/urdf/plastun.urdf (robot description, URDF)
Before this commit: robot MRC_"Plastun", 14 links, 13 joints
Joints:
- joint turrel_sered _ turrel_vverh up-to-down: axis 0  0  0 -> 0  1  0; limit lower=0 upper=0 effort=0 velocity=0 -> lower=-1 upper=1 effort=10 velocity=100; type fixed -> revolute
- joint turrel_vniz _ turrel_sered revolute: axis 0  0  0 -> 0  0  1; limit lower=0 upper=0 effort=0 velocity=0 -> lower=-5 upper=5 effort=2 velocity=100; type fixed -> revolute
- joint wheel_lev_1: limit lower=0.0 upper=0.548 effort=1000.0 velocity=0.5 -> lower=-1e+50 upper=1e+50 effort=-1 velocity=100
- joint wheel_lev_2: limit lower=0.0 upper=0.548 effort=1000.0 velocity=0.5 -> lower=-1e+50 upper=1e+50 effort=-1 velocity=100
- joint wheel_lev_3: limit lower=0.0 upper=0.548 effort=1000.0 velocity=0.5 -> lower=-1e+50 upper=1e+50 effort=-1 velocity=100
- joint wheel_prav_1: limit lower=0.0 upper=0.548 effort=1000.0 velocity=0.5 -> lower=-1e+50 upper=1e+50 effort=-1 velocity=100
- joint wheel_prav_2: limit lower=0.0 upper=0.548 effort=1000.0 velocity=0.5 -> lower=-1e+50 upper=1e+50 effort=-1 velocity=100
- joint wheel_prav_3: limit lower=0.0 upper=0.548 effort=1000.0 velocity=0.5 -> lower=-1e+50 upper=1e+50 effort=-1 velocity=100

Commit message: Исправлены часть недочетов, приложен gv, с графом соединений в роботе

File: plastun_description/urdf/plastun.urdf (robot description, URDF)
Before this commit: robot MRC_"Plastun", 14 links, 13 joints
Links:
- link camera_1: geometry collision mesh filename=package://plastun_description/meshes/STL_min/camera.stl scale=1 1 1; visual mesh filename=package://plastun_description/meshes/STL_min/camera.stl scale=1 1 1
- link camera_2: geometry collision mesh filename=package://plastun_description/meshes/STL_min/camera.stl scale=1 1 1; visual mesh filename=package://plastun_description/meshes/STL_min/camera.stl scale=1 1 1
Joints:
- joint turrel_sered _ turrel_vverh up-to-down: limit lower=-1 upper=1 effort=10 velocity=100 -> lower=-1 upper=1 effort=1 velocity=100; origin xyz=0.00306  0.00468  0.13878 rpy=0   0   0 -> xyz=0.00306  0.00468  0.12878 rpy=0   0   0

Commit message: Исправлена модель, добавлены сенсоры, покрашена модель для rviz

File: plastun_description/urdf/plastun.urdf (robot description, URDF)
Before this commit: robot MRC_"Plastun", 14 links, 13 joints
Links:
- added link base_link
Joints:
- added joint base_link_to_chassis: type fixed, parent base_link, child chassis
- joint camera_1 _ lazer_ukazka fixed: type fixed -> revolute
- joint chassis _ hokuyo fixed: type fixed -> revolute
- joint turrel_sered _ turrel_vverh up-to-down: type revolute -> fixed
- joint turrel_vverh _ camera_1 fixed: type fixed -> revolute
- joint turrel_vverh _ camera_2 fixed: type fixed -> revolute

Commit message: Добавлены сервоприводы, частично настроены моменты инерции, их стоит доделать

File: plastun_description/urdf/plastun.urdf (robot description, URDF)
Before this commit: robot MRC_Plastun, 15 links, 14 joints
Links:
- link camera_1: mass 0.0290342 -> 0.001
- link camera_2: mass 0.00092334 -> 0.003
- link hokuyo: mass 0.00014924 -> 0.3
- link lazer_ukazka: mass 0.5 -> 0.001
Joints:
- removed joint camera_1 _ lazer_ukazka fixed
- removed joint chassis _ hokuyo fixed
- removed joint chassis _ turrel_vniz fixed
- removed joint turrel_sered _ turrel_vverh up-to-down
- removed joint turrel_vniz _ turrel_sered revolute
- removed joint turrel_vverh _ camera_1 fixed
- removed joint turrel_vverh _ camera_2 fixed
- added joint camera_1_lazer_ukazka_fixed: type revolute, parent camera_1, child lazer_ukazka, origin xyz=-0.04766  0.00111  0.10548 rpy=0       0      0, axis 0  0  0, limit lower=0 upper=0 effort=0 velocity=0
- added joint chassis_hokuyo_fixed: type revolute, parent chassis, child hokuyo, origin xyz=0.15582  0.0808   0.42783 rpy=0       0       0, axis 0  0  0, limit lower=0 upper=0 effort=0 velocity=0
- added joint chassis_turrel_vniz_fixed: type fixed, parent chassis, child turrel_vniz, origin xyz=0.25857 -0.01238  0.42994 rpy=0 0  0, axis 0  0  0, limit lower=0 upper=0 effort=0 velocity=0
- added joint turrel_sered_turrel_vverh_up_to_down: type revolute, parent turrel_sered, child turrel_vverh, origin xyz=0.00306  0.00468  0.12878 rpy=0   0   0, axis 0  1  0, limit lower=-1 upper=1 effort=1 velocity=100
- added joint turrel_vniz_turrel_sered_revolute: type revolute, parent turrel_vniz, child turrel_sered, origin xyz=0.00045 -0.00033  0.13474 rpy=0  0   0, axis 0  0  1, limit lower=0 upper=0 effort=0 velocity=100
- added joint turrel_vverh_camera_1_ixed: type revolute, parent turrel_vverh, child camera_1, origin xyz=-0.07152 -0.21215 -0.017 rpy=0       0       0, axis 0  0  0, limit lower=0 upper=0 effort=0 velocity=0
- added joint turrel_vverh_camera_2_fixed: type revolute, parent turrel_vverh, child camera_2, origin xyz=-0.07152  0.21176 -0.017 rpy=0       0       0, axis 0  0  0, limit lower=0 upper=0 effort=0 velocity=0
