Commit message: Иправление координат модели

File: plastun_description/urdf/plastun.xacro (robot description, xacro)
@@ -8,6 +8,6 @@
   <xacro:property name="mass_wheels" value="1" />
   <xacro:property name="y_wheel" value="0.20499" />
-  <xacro:property name="z_wheel" value=" 0.15237" />
-  <xacro:property name="between_wheels" value="0.205" />
+  <xacro:property name="z_wheel" value=" 0.0925" />
+  <xacro:property name="between_wheels" value="0.2213343" />
   <xacro:property name="x_camera" value="-0.07152" />
   <xacro:property name="y_camera" value="0.21176" />
@@ -36,5 +36,5 @@
       <parent link="chassis"/>
       <child link="wheel_${prefix}_${num}"/>
-      <origin rpy="0       0      0" xyz="${0.13874 + (num - 1) * between_wheels} ${y_wheel * side}   ${z_wheel}"/>
+      <origin rpy="0       0      0" xyz="${0.1405513 + (num - 1) * between_wheels} ${y_wheel * side}   ${z_wheel}"/>
       <axis xyz="0 -1  0"/>
       <limit effort="-1" lower="-1e+50" upper="1e+50" velocity="100"/>
@@ -81,5 +81,5 @@
     </inertial>
     <collision >
-      <origin rpy="0  0  0" xyz="0.32045 0  0.06272"/>
+      <origin rpy="0  0  0" xyz="0 0  0"/>
       <geometry>
         <mesh filename="package://plastun_description/meshes/STL_min/chassis.stl" scale="1.0 1.0 1.0"/>
@@ -87,5 +87,5 @@
     </collision>
     <visual >
-      <origin rpy="0  0  0" xyz="0.32045 0  0.06272"/>
+      <origin rpy="0  0  0" xyz="0 0  0"/>
       <geometry>
         <mesh filename="package://plastun_description/meshes/STL_min/chassis.stl" scale="1 1 1"/>
@@ -216,5 +216,5 @@
     <parent link="chassis"/>
     <child link="hokuyo"/>
-    <origin rpy="0       0       0" xyz="0.15582  0.0808   0.42783"/>
+    <origin rpy="0       0       0" xyz="0.15586  0.083   0.365"/>
     <axis xyz="0  0  1"/>
     <limit effort="0" lower="0" upper="0" velocity="0"/>
@@ -223,5 +223,5 @@
     <parent link="chassis"/>
     <child link="turrel_vniz"/>
-    <origin rpy="0 0  0" xyz="0.25857 -0.01238  0.42994"/>
+    <origin rpy="0 0  0" xyz="0.255 0  0.37358"/>
     <axis xyz="0  0  0"/>
     <limit effort="0" lower="0" upper="0" velocity="0"/>
@@ -231,5 +231,5 @@
     <parent link="turrel_vniz"/>
     <child link="turrel_sered"/>
-    <origin rpy="0  0   0" xyz="0.00045 -0.00033  0.13474"/>
+    <origin rpy="0  0   0" xyz="0 0  0.13474"/>
     <axis xyz="0  0  1"/>
     <limit effort="0" lower="0" upper="0" velocity="100"/>
@@ -238,5 +238,5 @@
     <parent link="turrel_sered"/>
     <child link="turrel_vverh"/>
-    <origin rpy="0   0   0" xyz="0.00306  0.00468  0.1"/>
+    <origin rpy="0   0   0" xyz="0  0 0.1089254"/>
     <axis xyz="0  1  0"/>
     <limit effort="1" lower="-1" upper="1" velocity="100"/>

Commit message: Доисправлен xacro

File: plastun_description/urdf/plastun.xacro (robot description, xacro)
@@ -216,5 +216,5 @@
     <parent link="chassis"/>
     <child link="hokuyo"/>
-    <origin rpy="0       0       0" xyz="0.15586  0.083   0.365"/>
+    <origin rpy="0       0       0" xyz="0.14586  0.083   0.365"/>
     <axis xyz="0  0  1"/>
     <limit effort="0" lower="0" upper="0" velocity="0"/>
@@ -233,10 +233,10 @@
     <origin rpy="0  0   0" xyz="0 0  0.13474"/>
     <axis xyz="0  0  1"/>
-    <limit effort="0" lower="0" upper="0" velocity="100"/>
+    <limit effort="1" lower="-7" upper="7" velocity="10"/>
   </joint>
   <joint name="turrel_sered_turrel_vverh_up_to_down" type="revolute">
     <parent link="turrel_sered"/>
     <child link="turrel_vverh"/>
-    <origin rpy="0   0   0" xyz="0  0 0.1089254"/>
+    <origin rpy="0   0   0" xyz="0  0.005 0.1"/>
     <axis xyz="0  1  0"/>
     <limit effort="1" lower="-1" upper="1" velocity="100"/>

Commit message: Все детали имеют TF transform, исправлена модель, сделаны launch файлы для rviz в статике и, когда робот на карте

File: plastun_description/urdf/plastun.xacro (robot description, xacro)
@@ -1,305 +1,317 @@
 <?xml version="1.0"?>
 <robot name="MRC_Plastun" xmlns:xacro="http://www.ros.org/wiki/xacro">
-  <!-- Import all Gazebo-customization elements, including Gazebo colors -->
-  <xacro:include filename="$(find plastun_description)/urdf/plastun.gazebo" />
-  <!-- Import Rviz colors -->
-  <xacro:include filename="$(find rrbot_description)/urdf/materials.xacro" />
-  <!-- Constants for robot dimensions -->
-  <xacro:property name="mass_wheels" value="1" />
-  <xacro:property name="y_wheel" value="0.20499" />
-  <xacro:property name="z_wheel" value=" 0.0925" />
-  <xacro:property name="between_wheels" value="0.2213343" />
-  <xacro:property name="x_camera" value="-0.07152" />
-  <xacro:property name="y_camera" value="0.21176" />
-  <xacro:property name="z_camera" value="0" />
-  <xacro:macro name="wheel" params="prefix num side rev">
-    <link name="wheel_${prefix}_${num}">
-      <inertial>
-        <mass value="${mass_wheels}"/>
-        <origin rpy="0  0  0" xyz="0  0.000008  0"/>
-        <inertia ixx="0.166667" ixy="0" ixz="0" iyy="0.166667" iyz="0" izz="0.166667"/>
-      </inertial>
-      <collision >
-        <origin rpy="1.5708  0      0" xyz="0  0  0"/>
-        <geometry>
-          <cylinder length="0.09" radius="0.096"/>
-        </geometry>
-      </collision>
-      <visual>
-        <origin rpy="0  0  0" xyz="0  0  0"/>
-        <geometry>
-          <mesh filename="package://plastun_description/meshes/STL_min/wheel.stl" scale="1.0 1.0 1.0"/>
-        </geometry>
-      </visual>
-    </link>
-    <joint name="wheel_${rev}_${num}" type="revolute">
-      <parent link="chassis"/>
-      <child link="wheel_${prefix}_${num}"/>
-      <origin rpy="0       0      0" xyz="${0.1405513 + (num - 1) * between_wheels} ${y_wheel * side}   ${z_wheel}"/>
-      <axis xyz="0 -1  0"/>
-      <limit effort="-1" lower="-1e+50" upper="1e+50" velocity="100"/>
-    </joint>
-  </xacro:macro>
-  <xacro:macro name="camer" params="num side">
-    <link name="camera_${num}">
-      <inertial>
-        <mass value="0.001"/>
-        <origin rpy="0  0  0" xyz="-0.000018  -0.000225  0.060158"/>
-        <inertia ixx="0.00034961" ixy="0" ixz="0" iyy="0.00243426" iyz="0" izz="0.0027544"/>
-      </inertial>
-      <collision >
-        <origin rpy="0  0  0" xyz="0  0  0"/>
-        <geometry>
-          <mesh filename="package://plastun_description/meshes/STL_min/camera.stl" scale="1 1 1"/>
-        </geometry>
-      </collision>
-      <visual >
-        <origin rpy="0  0  0" xyz="0  0  0"/>
-        <geometry>
-          <mesh filename="package://plastun_description/meshes/STL_min/camera.stl" scale="1 1 1"/>
-        </geometry>
-      </visual>
-    </link>
-    <joint name="turrel_vverh_camera_${num}_fixed" type="revolute">
-      <parent link="turrel_vverh"/>
-      <child link="camera_${num}"/>
-      <origin rpy="0       0       0" xyz="${x_camera}  ${y_camera * side} ${z_camera}"/>
-      <axis xyz="0  0  1"/>
-      <limit effort="0" lower="0" upper="0" velocity="0"/>
-    </joint>
-  </xacro:macro>
-  <link name="base_link"/>
-  <joint name="base_link_to_chassis" type="fixed">
-    <parent link="base_link"/>
-    <child link="chassis"/>
-  </joint>
-  <link name="chassis">
-    <inertial>
-      <mass value="30"/>
-      <origin rpy="0  0  0" xyz="0.436419 -0.000612  0.228789"/>
-      <inertia ixx="0.166667" ixy="0" ixz="0" iyy="0.166667" iyz="0" izz="0.166667"/>
-    </inertial>
-    <collision >
-      <origin rpy="0  0  0" xyz="0 0  0"/>
-      <geometry>
-        <mesh filename="package://plastun_description/meshes/STL_min/chassis.stl" scale="1.0 1.0 1.0"/>
-      </geometry>
-    </collision>
-    <visual >
-      <origin rpy="0  0  0" xyz="0 0  0"/>
-      <geometry>
-        <mesh filename="package://plastun_description/meshes/STL_min/chassis.stl" scale="1 1 1"/>
-      </geometry>
-      <material name="green"/>
-    </visual>
-  </link>
-  <!--laser sensors -->
-  <link name="lazer_ukazka">
-    <inertial>
-      <mass value="0.001"/>
-      <origin rpy="0  0  0" xyz="-0.017806  0  0.027446"/>
-      <inertia ixx="0.0" ixy="0" ixz="0" iyy="0.0" iyz="0" izz="0.0"/>
-    </inertial>
-    <collision >
-      <origin rpy="0  0  0" xyz="0  0  0"/>
-      <geometry>
-        <mesh filename="package://plastun_description/meshes/STL_min/lazer_ukazka.stl" scale="1.0 1.0 1.0"/>
-      </geometry>
-    </collision>
-    <visual >
-      <origin rpy="0  0  0" xyz="0  0  0"/>
-      <geometry>
-        <mesh filename="package://plastun_description/meshes/STL_min/lazer_ukazka.stl" scale="1.0 1.0 1.0"/>
-      </geometry>
-      <material name="white"/>
-    </visual>
-  </link>
-  <link name="hokuyo">
-    <inertial>
-      <mass value="0.3"/>
-      <origin rpy="0  0  0" xyz="-0.000001  0  0.053927"/>
-      <inertia ixx="0.166667" ixy="0" ixz="0" iyy="0.166667" iyz="0" izz="0.166667"/>
-    </inertial>
-    <collision >
-      <origin rpy="0  0  0" xyz="0    0    0.05"/>
-      <geometry>
-        <box size="0.06524 0.079833 0.102579"/>
-      </geometry>
-    </collision>
-    <visual >
-      <origin rpy="0  0  0" xyz="0  0  0"/>
-      <geometry>
-        <mesh filename="package://plastun_description/meshes/STL_min/hokuyo.stl" scale="1 1 1"/>
-      </geometry>
-    </visual>
-  </link>
-  <!-- Turrel -->
-  <link name="turrel_vniz">
-    <inertial>
-      <mass value="1"/>
-      <origin rpy="0  0  0" xyz="-0.000002  0  0.072908"/>
-      <inertia ixx="0.166667" ixy="0" ixz="0" iyy="0.166667" iyz="0" izz="0.166667"/>
-    </inertial>
-    <collision >
-      <origin rpy="0  0  0" xyz="0  0  0"/>
-      <geometry>
-        <mesh filename="package://plastun_description/meshes/STL_min/turrel_vniz.stl" scale="1.0 1.0 1.0"/>
-      </geometry>
-    </collision>
-    <visual >
-      <origin rpy="0  0  0" xyz="0  0  0"/>
-      <geometry>
-        <mesh filename="package://plastun_description/meshes/STL_min/turrel_vniz.stl" scale="1.0 1.0 1.0"/>
-      </geometry>
-      <material name="white"/>
-    </visual>
-  </link>
-  <link name="turrel_sered">
-    <inertial>
-      <mass value="1"/>
-      <origin rpy="0  0  0" xyz="0  0  0.089664"/>
-      <inertia ixx="0.166667" ixy="0" ixz="0" iyy="0.166667" iyz="0" izz="0.166667"/>
-    </inertial>
-    <collision >
-      <origin rpy="0  0  0" xyz="0  0  0"/>
-      <geometry>
-        <mesh filename="package://plastun_description/meshes/STL_min/turrel_sered.stl" scale="1.0 1.0 1.0"/>
-      </geometry>
-    </collision>
-    <visual >
-      <origin rpy="0  0  0" xyz="0  0  0"/>
-      <geometry>
-        <mesh filename="package://plastun_description/meshes/STL_min/turrel_sered.stl" scale="1.0 1.0 1.0"/>
-      </geometry>
-      <material name="brown"/>
-    </visual>
-  </link>
-  <link name="turrel_vverh">
-    <inertial>
-      <mass value="1"/>
-      <origin rpy="0  0  0" xyz="0    -0.005000   0.051671"/>
-      <inertia ixx="0.166667" ixy="0" ixz="0" iyy="0.166667" iyz="0" izz="0.166667"/>
-    </inertial>
-    <collision >
-      <origin rpy="0  0  0" xyz="0    0   0"/>
-      <geometry>
-        <mesh filename="package://plastun_description/meshes/STL_min/turrel_vverh.stl" scale="1.0 1.0 1.0"/>
-      </geometry>
-    </collision>
-    <visual >
-      <origin rpy="0  0  0" xyz="0    0   0"/>
-      <geometry>
-        <mesh filename="package://plastun_description/meshes/STL_min/turrel_vverh.stl" scale="1.0 1.0 1.0"/>
-      </geometry>
-      <material name="blue"/>
-    </visual>
-  </link>
-  <!--cameras (links and joints(fix with turrel_verh)) -->
-  <xacro:camer num="1" side="-1"/>
-  <xacro:camer num="2" side="1"/>
-  <!-- wheels (links and joints(revolute, parrent - chassis))-->
-  <xacro:wheel prefix="left" num="1" side="-1" rev="lev"/>
-  <xacro:wheel prefix="left" num="2" side="-1" rev="lev"/>
-  <xacro:wheel prefix="left" num="3" side="-1" rev="lev"/>
-  <xacro:wheel prefix="right" num="1" side="1" rev="prav"/>
-  <xacro:wheel prefix="right" num="2" side="1" rev="prav"/>
-  <xacro:wheel prefix="right" num="3" side="1" rev="prav"/>
-  <!--fix'es joints -->
-  <joint name="camera_1_lazer_ukazka_fixed" type="revolute">
-    <parent link="camera_1"/>
-    <child link="lazer_ukazka"/>
-    <origin rpy="0       0      0" xyz="-0.04766  0.00111  0.10548"/>
-    <axis xyz="0  0  1"/>
-    <limit effort="0" lower="0" upper="0" velocity="0"/>
-  </joint>
-  <joint name="chassis_hokuyo_fixed" type="revolute">
-    <parent link="chassis"/>
-    <child link="hokuyo"/>
-    <origin rpy="0       0       0" xyz="0.14586  0.083   0.365"/>
-    <axis xyz="0  0  1"/>
-    <limit effort="0" lower="0" upper="0" velocity="0"/>
-  </joint>
-  <joint name="chassis_turrel_vniz_fixed" type="fixed">
-    <parent link="chassis"/>
-    <child link="turrel_vniz"/>
-    <origin rpy="0 0  0" xyz="0.255 0  0.37358"/>
-    <axis xyz="0  0  0"/>
-    <limit effort="0" lower="0" upper="0" velocity="0"/>
-  </joint>
-  <!-- revolute joints -->
-  <joint name="turrel_vniz_turrel_sered_revolute" type="revolute">
-    <parent link="turrel_vniz"/>
-    <child link="turrel_sered"/>
-    <origin rpy="0  0   0" xyz="0 0  0.13474"/>
-    <axis xyz="0  0  1"/>
-    <limit effort="1" lower="-7" upper="7" velocity="10"/>
-  </joint>
-  <joint name="turrel_sered_turrel_vverh_up_to_down" type="revolute">
-    <parent link="turrel_sered"/>
-    <child link="turrel_vverh"/>
-    <origin rpy="0   0   0" xyz="0  0.005 0.1"/>
-    <axis xyz="0  1  0"/>
-    <limit effort="1" lower="-1" upper="1" velocity="100"/>
-  </joint>
-  <!--transmitions-->
-  <transmission name="wheel_l_1">
-    <type>transmission_interface/SimpleTransmission</type>
-    <joint name="wheel_lev_1">
-      <hardwareInterface>EffortJointInterface</hardwareInterface>
-    </joint>
-    <actuator name="wh_l_1">
-      <hardwareInterface>EffortJointInterface</hardwareInterface>
-      <mechanicalReduction>1</mechanicalReduction>
-    </actuator>
-  </transmission>
-  <transmission name="wheel_l_3">
-    <type>transmission_interface/SimpleTransmission</type>
-    <joint name="wheel_lev_3">
-      <hardwareInterface>EffortJointInterface</hardwareInterface>
-    </joint>
-    <actuator name="wh_l_3">
-      <hardwareInterface>EffortJointInterface</hardwareInterface>
-      <mechanicalReduction>1</mechanicalReduction>
-    </actuator>
-  </transmission>
-  <transmission name="wheel_r_1">
-    <type>transmission_interface/SimpleTransmission</type>
-    <joint name="wheel_prav_1">
-      <hardwareInterface>EffortJointInterface</hardwareInterface>
-    </joint>
-    <actuator name="wh_r_1">
-      <hardwareInterface>EffortJointInterface</hardwareInterface>
-      <mechanicalReduction>1</mechanicalReduction>
-    </actuator>
-  </transmission>
-  <transmission name="wheel_r_3">
-    <type>transmission_interface/SimpleTransmission</type>
-    <joint name="wheel_prav_3">
-      <hardwareInterface>EffortJointInterface</hardwareInterface>
-    </joint>
-    <actuator name="wh_r_3">
-      <hardwareInterface>EffortJointInterface</hardwareInterface>
-      <mechanicalReduction>1</mechanicalReduction>
-    </actuator>
-  </transmission>
-  <transmission name="turrel_revol">
-    <type>transmission_interface/SimpleTransmission</type>
-    <joint name="turrel_vniz_turrel_sered_revolute">
-      <hardwareInterface>EffortJointInterface</hardwareInterface>
-    </joint>
-    <actuator name="tl_rev">
-      <hardwareInterface>EffortJointInterface</hardwareInterface>
-      <mechanicalReduction>1</mechanicalReduction>
-    </actuator>
-  </transmission>
-  <transmission name="turrel_up_to_down">
-    <type>transmission_interface/SimpleTransmission</type>
-    <joint name="turrel_sered_turrel_vverh_up_to_down">
-      <hardwareInterface>EffortJointInterface</hardwareInterface>
-    </joint>
-    <actuator name="tl_ud">
-      <hardwareInterface>EffortJointInterface</hardwareInterface>
-      <mechanicalReduction>1</mechanicalReduction>
-    </actuator>
-  </transmission>
+	<!-- Import all Gazebo-customization elements, including Gazebo colors -->
+	<xacro:include filename="$(find plastun_description)/urdf/plastun.gazebo" />
+	<!-- Import Rviz colors -->
+	<xacro:include filename="$(find rrbot_description)/urdf/materials.xacro" />
+	<!-- Constants for robot dimensions -->
+	<xacro:property name="mass_wheels" value="1" />
+	<xacro:property name="y_wheel" value="0.20499" />
+	<xacro:property name="z_wheel" value=" 0.0925" />
+	<xacro:property name="between_wheels" value="0.2213343" />
+	<xacro:property name="x_camera" value="-0.07152" />
+	<xacro:property name="y_camera" value="0.21176" />
+	<xacro:property name="z_camera" value="0" />
+	<xacro:macro name="wheel" params="prefix num side rev">
+		<link name="wheel_${prefix}_${num}">
+			<inertial>
+				<mass value="${mass_wheels}"/>
+				<origin rpy="0  0  0" xyz="0  0.000008  0"/>
+				<inertia ixx="0.166667" ixy="0" ixz="0" iyy="0.166667" iyz="0" izz="0.166667"/>
+			</inertial>
+			<collision >
+				<origin rpy="1.5708  0      0" xyz="0  0  0"/>
+				<geometry>
+					<cylinder length="0.09" radius="0.096"/>
+				</geometry>
+			</collision>
+			<visual>
+				<origin rpy="0  0  0" xyz="0  0  0"/>
+				<geometry>
+					<mesh filename="package://plastun_description/meshes/STL_min/wheel.stl" scale="1.0 1.0 1.0"/>
+				</geometry>
+			</visual>
+		</link>
+		<joint name="wheel_${rev}_${num}" type="revolute">
+			<parent link="chassis"/>
+			<child link="wheel_${prefix}_${num}"/>
+			<origin rpy="0       0      0" xyz="${0.1405513 + (num - 1) * between_wheels} ${y_wheel * side}   ${z_wheel}"/>
+			<axis xyz="0 -1  0"/>
+			<limit effort="-1" lower="-1e+50" upper="1e+50" velocity="100"/>
+		</joint>
+	</xacro:macro>
+	<xacro:macro name="transmission_wheel" params="rev num side_name">
+		<transmission name="wheel_${side_name}_${num}">
+			<type>transmission_interface/SimpleTransmission</type>
+			<joint name="wheel_${rev}_${num}">
+				<hardwareInterface>EffortJointInterface</hardwareInterface>
+			</joint>
+			<actuator name="wh_${side_name}_${num}">
+				<hardwareInterface>EffortJointInterface</hardwareInterface>
+				<mechanicalReduction>1</mechanicalReduction>
+			</actuator>
+		</transmission>
+	</xacro:macro>
+	<xacro:macro name="camer" params="num side">
+		<link name="camera_${num}">
+			<inertial>
+				<mass value="0.001"/>
+				<origin rpy="0  0  0" xyz="-0.000018  -0.000225  0.060158"/>
+				<inertia ixx="0.00034961" ixy="0" ixz="0" iyy="0.00243426" iyz="0" izz="0.0027544"/>
+			</inertial>
+			<collision >
+				<origin rpy="0  0  0" xyz="0  0  0"/>
+				<geometry>
+					<mesh filename="package://plastun_description/meshes/STL_min/camera.stl" scale="1 1 1"/>
+				</geometry>
+			</collision>
+			<visual >
+				<origin rpy="0  0  0" xyz="0  0  0"/>
+				<geometry>
+					<mesh filename="package://plastun_description/meshes/STL_min/camera.stl" scale="1 1 1"/>
+				</geometry>
+			</visual>
+		</link>
+		<joint name="turrel_vverh_camera_${num}_fixed" type="revolute">
+			<parent link="turrel_vverh"/>
+			<child link="camera_${num}"/>
+			<origin rpy="0       0       0" xyz="${x_camera}  ${y_camera * side} ${z_camera}"/>
+			<axis xyz="0  0  1"/>
+			<limit effort="0" lower="0" upper="0" velocity="0"/>
+		</joint>
+	</xacro:macro>
+	<xacro:macro name="transmission_camera" params="num">
+		<transmission name="camer_${num}">
+			<type>transmission_interface/SimpleTransmission</type>
+			<joint name="turrel_vverh_camera_${num}_fixed">
+				<hardwareInterface>EffortJointInterface</hardwareInterface>
+			</joint>
+			<actuator name="cam_${num}">
+				<hardwareInterface>EffortJointInterface</hardwareInterface>
+				<mechanicalReduction>1</mechanicalReduction>
+			</actuator>
+		</transmission>
+	</xacro:macro>
+	<link name="base_link"/>
+	<joint name="chassis_base_link_fixed" type="fixed">
+		<parent link="base_link"/>
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
File: plastun_description/urdf/plastun_generated.urdf (robot description, URDF)
Before this commit: robot MRC_Plastun, 15 links, 14 joints
Joints:
- removed joint base_link_to_chassis
- added joint chassis_base_link_fixed: type fixed, parent base_link, child chassis
- joint chassis_hokuyo_fixed: origin xyz=0.15582  0.0808   0.42783 rpy=0       0       0 -> xyz=0.14586  0.083   0.365 rpy=0       0       0
- joint chassis_turrel_vniz_fixed: origin xyz=0.25857 -0.01238  0.42994 rpy=0 0  0 -> xyz=0.255 0  0.37358 rpy=0 0  0
- joint turrel_sered_turrel_vverh_up_to_down: origin xyz=0.00306  0.00468  0.1 rpy=0   0   0 -> xyz=0  0.005 0.1 rpy=0   0   0
- joint turrel_vniz_turrel_sered_revolute: limit lower=0 upper=0 effort=0 velocity=100 -> lower=-7 upper=7 effort=1 velocity=10; origin xyz=0.00045 -0.00033  0.13474 rpy=0  0   0 -> xyz=0 0  0.13474 rpy=0  0   0
- joint wheel_lev_1: origin xyz=0.13874 -0.20499   0.15237 rpy=0       0      0 -> xyz=0.1405513 -0.20499   0.0925 rpy=0       0      0
- joint wheel_lev_2: origin xyz=0.34374 -0.20499   0.15237 rpy=0       0      0 -> xyz=0.3618856 -0.20499   0.0925 rpy=0       0      0
- joint wheel_lev_3: origin xyz=0.54874 -0.20499   0.15237 rpy=0       0      0 -> xyz=0.5832199 -0.20499   0.0925 rpy=0       0      0
- joint wheel_prav_1: origin xyz=0.13874 0.20499   0.15237 rpy=0       0      0 -> xyz=0.1405513 0.20499   0.0925 rpy=0       0      0
- joint wheel_prav_2: origin xyz=0.34374 0.20499   0.15237 rpy=0       0      0 -> xyz=0.3618856 0.20499   0.0925 rpy=0       0      0
- joint wheel_prav_3: origin xyz=0.54874 0.20499   0.15237 rpy=0       0      0 -> xyz=0.5832199 0.20499   0.0925 rpy=0       0      0
