Commit message: Модель работает на 6и колесах, вращение и трения в норме, на ближайшее время изменять не требуется, опытным путем макс скорость 3.0, мин поворот 1.9 макс поворот 5

File: plastun_description/urdf/plastun.xacro (robot description, xacro)
@@ -22,5 +22,5 @@
 	<xacro:property name="y_camera" value="0.21" />
 	<xacro:property name="z_camera" value="0.003" />
-	<xacro:macro name="wheel" params="prefix num side rev">
+	<xacro:macro name="wheel" params="prefix num side rev collision">
 		<link name="wheel_${prefix}_${num}">
 			<inertial>
@@ -29,4 +29,5 @@
 				<inertia ixx="0.000000000" ixy="0" ixz="0" iyy="0.000000000" iyz="0" izz="0.000000000"/>
 			</inertial>
+	<xacro:if value="${collision == 1}">
 			<collision >
 				<origin rpy="1.5708  0      0" xyz="0  0  0"/>
@@ -35,4 +36,5 @@
 				</geometry>
 			</collision>
+	</xacro:if>
 			<visual>
 				<origin rpy="0  0  0" xyz="0  0  0"/>
@@ -50,5 +52,6 @@
 		</joint>
 	</xacro:macro>
-	<xacro:macro name="transmission_wheel" params="rev num side_name">
+	<xacro:macro name="transmission_wheel" params="rev num side_name collision">
+	<xacro:if value="${collision == 1}">
 		<transmission name="wheel_${side_name}_${num}">
 			<type>transmission_interface/SimpleTransmission</type>
@@ -61,4 +64,5 @@
 			</actuator>
 		</transmission>
+	</xacro:if>
 	</xacro:macro>
 	<xacro:macro name="camer" params="num side">
@@ -208,10 +212,10 @@
 	<xacro:camer num="2" side="-1"/>
 	<!-- wheels (links and joints(revolute, parrent - chassis))-->
-	<xacro:wheel prefix="left" num="1" side="1" rev="lev"/>
-	<xacro:wheel prefix="left" num="2" side="1" rev="lev"/>
-	<xacro:wheel prefix="left" num="3" side="1" rev="lev"/>
-	<xacro:wheel prefix="right" num="1" side="-1" rev="prav"/>
-	<xacro:wheel prefix="right" num="2" side="-1" rev="prav"/>
-	<xacro:wheel prefix="right" num="3" side="-1" rev="prav"/>
+	<xacro:wheel prefix="left" num="1" side="1" rev="lev" collision="1"/>
+	<xacro:wheel prefix="left" num="2" side="1" rev="lev" collision="1"/>
+	<xacro:wheel prefix="left" num="3" side="1" rev="lev" collision="1"/>
+	<xacro:wheel prefix="right" num="1" side="-1" rev="prav" collision="1"/>
+	<xacro:wheel prefix="right" num="2" side="-1" rev="prav" collision="1"/>
+	<xacro:wheel prefix="right" num="3" side="-1" rev="prav" collision="1"/>
 	<!--fix'es joints -->
 	<joint name="camera_1_lazer_ukazka_fixed" type="fixed">
@@ -242,5 +246,5 @@
 		<origin rpy="0  0   0" xyz="0 0  0.1296088"/>
 		<axis xyz="0  0  1"/>
-		<limit effort="1" lower="-7" upper="7" velocity="10"/>
+		<limit effort="1" lower="-3.139" upper="3.139" velocity="100"/>
 	</joint>
 	<joint name="turrel_sered_turrel_vverh_up_to_down" type="revolute">
@@ -272,9 +276,9 @@
 		</actuator>
 	</transmission>
-	<xacro:transmission_wheel num="1" side_name="l" rev="lev"/>
-	<xacro:transmission_wheel num="2" side_name="l" rev="lev"/>
-	<xacro:transmission_wheel num="3" side_name="l" rev="lev"/>
-	<xacro:transmission_wheel num="1" side_name="r" rev="prav"/>
-	<xacro:transmission_wheel num="2" side_name="r" rev="prav"/>
-	<xacro:transmission_wheel num="3" side_name="r" rev="prav"/>
+	<xacro:transmission_wheel num="1" side_name="l" rev="lev" collision="1"/>
+	<xacro:transmission_wheel num="2" side_name="l" rev="lev" collision="1"/>
+	<xacro:transmission_wheel num="3" side_name="l" rev="lev" collision="1"/>
+	<xacro:transmission_wheel num="1" side_name="r" rev="prav" collision="1"/>
+	<xacro:transmission_wheel num="2" side_name="r" rev="prav" collision="1"/>
+	<xacro:transmission_wheel num="3" side_name="r" rev="prav" collision="1"/>
 </robot>

Commit message: Добавлен плафон как цель, улучшена модель и исправлены характеристи в base_local_scanner и costmap config

File: plastun_description/urdf/plastun.xacro (robot description, xacro)
@@ -25,5 +25,5 @@
 		<link name="wheel_${prefix}_${num}">
 			<inertial>
-				<mass value="2"/>
+				<mass value="0.03"/>
 				<origin rpy="0  0  0" xyz="0  0.000007723  0"/>
 				<inertia ixx="0.000000000" ixy="0" ixz="0" iyy="0.000000000" iyz="0" izz="0.000000000"/>
@@ -213,8 +213,8 @@
 	<!-- wheels (links and joints(revolute, parrent - chassis))-->
 	<xacro:wheel prefix="left" num="1" side="1" rev="lev" collision="1"/>
-	<xacro:wheel prefix="left" num="2" side="1" rev="lev" collision="1"/>
+	<xacro:wheel prefix="left" num="2" side="1" rev="lev" collision="0"/>
 	<xacro:wheel prefix="left" num="3" side="1" rev="lev" collision="1"/>
 	<xacro:wheel prefix="right" num="1" side="-1" rev="prav" collision="1"/>
-	<xacro:wheel prefix="right" num="2" side="-1" rev="prav" collision="1"/>
+	<xacro:wheel prefix="right" num="2" side="-1" rev="prav" collision="0"/>
 	<xacro:wheel prefix="right" num="3" side="-1" rev="prav" collision="1"/>
 	<!--fix'es joints -->
