Commit message: Проведены работы над ошибками, исправлен general_targeting, прописаны зависимости для global_control_system

File: plastun_description/urdf/plastun_generated.urdf (robot description, URDF)
Before this commit: robot MRC_Plastun, 15 links, 14 joints
Links:
- link wheel_left_1: mass 2 -> 0.03
- link wheel_left_2: mass 2 -> 0.03; geometry visual mesh filename=package://plastun_description/meshes/STL_min/wheel.stl scale=1.0 1.0 1.0
- link wheel_left_3: mass 2 -> 0.03
- link wheel_right_1: mass 2 -> 0.03
- link wheel_right_2: mass 2 -> 0.03; geometry visual mesh filename=package://plastun_description/meshes/STL_min/wheel.stl scale=1.0 1.0 1.0
- link wheel_right_3: mass 2 -> 0.03
Joints:
- joint turrel_sered_turrel_vverh_up_to_down: axis 0  1  0 -> 0  -1  0
- joint turrel_vniz_turrel_sered_revolute: limit lower=-7 upper=7 effort=1 velocity=10 -> lower=-3.139 upper=3.139 effort=1 velocity=100
- joint turrel_vverh_camera_1_fixed: origin xyz=0.2  -0.21 0.0576695 rpy=0       0       0 -> xyz=0.2  0.21 0.0576695 rpy=0       0       0
- joint turrel_vverh_camera_2_fixed: origin xyz=0.2  0.21 0.0576695 rpy=0       0       0 -> xyz=0.2  -0.21 0.0576695 rpy=0       0       0
- joint wheel_lev_1: limit lower=-1e+50 upper=1e+50 effort=-1 velocity=100 -> lower=-1e+100 upper=1e+100 effort=-1 velocity=100; origin xyz=0.0666644 -0.20499   0.096 rpy=0       0      0 -> xyz=0.0666644 0.20499   0.096 rpy=0       0      0
- joint wheel_lev_2: limit lower=-1e+50 upper=1e+50 effort=-1 velocity=100 -> lower=-1e+100 upper=1e+100 effort=-1 velocity=100; origin xyz=0.2881144 -0.20499   0.096 rpy=0       0      0 -> xyz=0.2881144 0.20499   0.096 rpy=0       0      0
- joint wheel_lev_3: limit lower=-1e+50 upper=1e+50 effort=-1 velocity=100 -> lower=-1e+100 upper=1e+100 effort=-1 velocity=100; origin xyz=0.5095644 -0.20499   0.096 rpy=0       0      0 -> xyz=0.5095644 0.20499   0.096 rpy=0       0      0
- joint wheel_prav_1: limit lower=-1e+50 upper=1e+50 effort=-1 velocity=100 -> lower=-1e+100 upper=1e+100 effort=-1 velocity=100; origin xyz=0.0666644 0.20499   0.096 rpy=0       0      0 -> xyz=0.0666644 -0.20499   0.096 rpy=0       0      0
- joint wheel_prav_2: limit lower=-1e+50 upper=1e+50 effort=-1 velocity=100 -> lower=-1e+100 upper=1e+100 effort=-1 velocity=100; origin xyz=0.2881144 0.20499   0.096 rpy=0       0      0 -> xyz=0.2881144 -0.20499   0.096 rpy=0       0      0
- joint wheel_prav_3: limit lower=-1e+50 upper=1e+50 effort=-1 velocity=100 -> lower=-1e+100 upper=1e+100 effort=-1 velocity=100; origin xyz=0.5095644 0.20499   0.096 rpy=0       0      0 -> xyz=0.5095644 -0.20499   0.096 rpy=0       0      0
